Commit message: Integrated Lidar to simulation (needs tuning to spec before attempting odom)

File: catkin_ws/src/robot_description/urdf/robot.urdf (robot description, URDF)
Before this commit: robot myAGV, 2 links, 1 joints
Links:
- added link lidar_link, mass 0.1; collision cylinder length=0.04 radius=0.05; visual cylinder length=0.04 radius=0.05
- link base_footprint: mass None -> 1.0; geometry collision box size=0.4 0.3 0.1; visual mesh filename=package://robot_description/urdf/myagv_base.dae scale=1 1 1
- link base_up: mass None -> 0.5; geometry collision box size=0.3 0.3 0.2; visual mesh filename=package://robot_description/urdf/myagv_up.dae scale=1 1 1
Joints:
- added joint lidar_joint: type fixed, parent base_up, child lidar_link, origin xyz=0.0 0.0 0.2 rpy=0 0 0
