Commit message: urdf fix

File: catkin_ws/src/robot_description/urdf/assembly.urdf (robot description, URDF)
Before this commit: robot myagv_assembly, 4 links, 3 joints
Links:
- removed link camera_mount_link
- link base_link: geometry visual mesh filename=package://robot_description/meshes/stl/assembly.stl scale=0.001 0.001 0.001
- link camera_link: geometry 
Joints:
- removed joint camera_mount_joint

Commit message: tf links fix 1.0

File: catkin_ws/src/robot_description/urdf/assembly.urdf (robot description, URDF)
Before this commit: robot myagv_assembly, 3 links, 2 joints
Links:
- added link lidar_link
- added link mount_link
Joints:
- added joint lidar_joint: type fixed, parent base_link, child lidar_link, origin xyz=0 0 0 rpy=0 0 0
- added joint mount_joint: type fixed, parent base_link, child mount_link, origin xyz=-0.269921 0.156212 -0.093832 rpy=-3.133687 0 3.141593

Commit message: changed mount joint

File: catkin_ws/src/robot_description/urdf/assembly.urdf (robot description, URDF)
Before this commit: robot myagv_assembly, 5 links, 4 joints
Joints:
- joint camera_joint: parent base_link -> mount_link

Commit message: tf links fix 2.0

File: catkin_ws/src/robot_description/urdf/assembly.urdf (robot description, URDF)
Before this commit: robot myagv_assembly, 5 links, 4 joints
Joints:
- joint camera_joint: origin xyz=-0.300426 0.226662 -0.100389 rpy=-3.133687 0 3.141593 -> xyz=0.030505 0.070500 0.006000 rpy=0 0 0; parent base_link -> mount_link
- joint mount_joint: origin xyz=-0.269921 0.156212 -0.093832 rpy=-3.133687 0 3.141593 -> xyz=-0.269921 0.093832 0.156212 rpy=1.578702 0 3.141593

Commit message: tf links fix 3.0

File: catkin_ws/src/robot_description/urdf/assembly.urdf (robot description, URDF)
Before this commit: robot myagv_assembly, 5 links, 4 joints
Joints:
- joint camera_joint: origin xyz=0.030505 0.070500 0.006000 rpy=0 0 0 -> xyz=0.000505 -0.057000 0.023000 rpy=0 0 0
- joint mount_joint: origin xyz=-0.269921 0.093832 0.156212 rpy=1.578702 0 3.141593 -> xyz=-0.299921 0.064841 0.283945 rpy=1.578702 0 3.141593

Commit message: tf links fix 4.0

File: catkin_ws/src/robot_description/urdf/assembly.urdf (robot description, URDF)
Before this commit: robot myagv_assembly, 5 links, 4 joints
Links:
- added link base_footprint
Joints:
- added joint base_footprint_to_base_link: type fixed, parent base_footprint, child base_link, origin xyz=0 0 0.23 rpy=0 0 0
- joint camera_joint: origin xyz=0.000505 -0.057000 0.023000 rpy=0 0 0 -> xyz=0.030505 0.070500 0.006000 rpy=0 0 0
- joint mount_joint: origin xyz=-0.299921 0.064841 0.283945 rpy=1.578702 0 3.141593 -> xyz=-0.269921 0.093832 0.156212 rpy=1.578702 0 3.141593

Commit message: tf links fix 5.0

File: catkin_ws/src/robot_description/urdf/assembly.urdf (robot description, URDF)
Before this commit: robot myagv_assembly, 6 links, 5 joints
Links:
- removed link base_footprint
Joints:
- removed joint base_footprint_to_base_link
- joint mount_joint: origin xyz=-0.269921 0.093832 0.156212 rpy=1.578702 0 3.141593 -> xyz=0.030075 0.126506 -0.073735 rpy=1.578702 0 3.141593

Commit message: tf links fix 6.0

File: catkin_ws/src/robot_description/urdf/assembly.urdf (robot description, URDF)
Before this commit: robot myagv_assembly, 5 links, 4 joints
Links:
- added link myagv_link; visual mesh filename=package://robot_description/meshes/stl/assembly.stl scale=0.001 0.001 0.001
- added link odom_link
- link base_link: geometry 
Joints:
- added joint base_to_lidar: type fixed, parent base_link, child lidar_link, origin xyz=0 0 0 rpy=0 0 0
- added joint base_to_myagv: type fixed, parent base_link, child myagv_link, origin xyz=0.049350 -0.012983 -0.117401 rpy=0 0 0
- added joint base_to_odom: type fixed, parent base_link, child odom_link, origin xyz=0 0 0 rpy=0 0 0
- joint mount_joint: origin xyz=0.030075 0.126506 -0.073735 rpy=1.578702 0 3.141593 -> xyz=-0.220571 0.143229 -0.211233 rpy=-3.133687 0 3.141593

Commit message: tf links fix 7.0 - should work

File: catkin_ws/src/robot_description/urdf/assembly.urdf (robot description, URDF)
Before this commit: robot myagv_assembly, 7 links, 7 joints
Joints:
- removed joint lidar_joint
- joint base_to_myagv: origin xyz=0.049350 -0.012983 -0.117401 rpy=0 0 0 -> xyz=-0.018406 0.295891 -0.159293 rpy=1.578702 0.007906 1.570796
- joint mount_joint: origin xyz=-0.220571 0.143229 -0.211233 rpy=-3.133687 0 3.141593 -> xyz=-0.111000 0.027219 -0.000215 rpy=1.570796 -0.007906 -1.570796

Commit message: fixed transforms and launch files

File: catkin_ws/src/robot_description/urdf/assembly.urdf (robot description, URDF)
Before this commit: robot myagv_assembly, 7 links, 6 joints
Links:
- removed link lidar_link
- removed link odom_link
- added link mocap_link
Joints:
- removed joint base_to_lidar
- removed joint base_to_odom
- added joint base_to_mocap: type fixed, parent base_link, child mocap_link, origin xyz=0 0 0 rpy=0 0 0
- joint base_to_myagv: origin xyz=-0.018406 0.295891 -0.159293 rpy=1.578702 0.007906 1.570796 -> xyz=-0.018406 0.295891 0.159293 rpy=1.578702 0.007906 1.570796

Commit message: urdf adjustment base_link

File: catkin_ws/src/robot_description/urdf/assembly.urdf (robot description, URDF)
Before this commit: robot myagv_assembly, 6 links, 5 joints
Joints:
- joint base_to_myagv: origin xyz=-0.018406 0.295891 0.159293 rpy=1.578702 0.007906 1.570796 -> xyz=-0.018406 0.295891 -0.159293 rpy=1.578702 0.007906 1.570796

Commit message: fixed assembly (set z to 0)

File: catkin_ws/src/robot_description/urdf/assembly.urdf (robot description, URDF)
Before this commit: robot myagv_assembly, 8 links, 7 joints
Joints:
- joint base_to_led_marker: origin xyz=-0.015025 0.002880 -0.000023 rpy=0 0 0 -> xyz=-0.015025 0.002880 0.117401 rpy=0 0 0
- joint base_to_myagv: origin xyz=-0.033431 0.298771 -0.159316 rpy=1.578702 0.007906 1.570796 -> xyz=-0.033431 0.298771 -0.041892 rpy=1.578702 0.007906 1.570796
- joint mount_joint: origin xyz=-0.126025 0.030099 -0.000238 rpy=1.570796 -0.007906 -1.570796 -> xyz=-0.126025 0.030099 0.117186 rpy=1.570796 -0.007906 -1.570796

Commit message: submodules merging

File: catkin_ws/src/robot_description/urdf/assembly.urdf (robot description, URDF)
Before this commit: robot myagv_assembly, 8 links, 7 joints
Links:
- removed link led_marker_link
- removed link mount_link
- removed link myagv_link
- removed link odom_link
- added link assembly_mesh_link; visual mesh filename=package://robot_description/meshes/stl/assembly.stl scale=0.001 0.001 0.001
- added link base_footprint
- added link camera_color_frame
- added link camera_color_optical_frame
- added link camera_depth_frame
- added link camera_depth_optical_frame
- added link laser_frame; visual cylinder length=0.05 radius=0.035
- added link mocap_led_0; visual sphere radius=0.012
- added link mocap_led_1; visual sphere radius=0.012
- added link mocap_led_2; visual sphere radius=0.012
- added link mocap_led_3; visual sphere radius=0.012
- added link mocap_led_4; visual sphere radius=0.012
- added link mocap_led_5; visual sphere radius=0.012
- added link mocap_led_6; visual sphere radius=0.012
- added link mocap_led_7; visual sphere radius=0.012
- link camera_link: geometry visual box size=0.095 0.025 0.025
Joints:
- removed joint base_to_led_marker
- removed joint base_to_lidar
- removed joint base_to_myagv
- removed joint base_to_odom
- removed joint camera_joint
- removed joint camera_optical_joint
- removed joint mount_joint
- added joint base_footprint_to_base_link: type fixed, parent base_footprint, child base_link, origin xyz=0 0 0 rpy=0 0 0
- added joint base_to_assembly_mesh: type fixed, parent base_link, child assembly_mesh_link, origin xyz=0.299832 -0.024717 -0.033859 rpy=0 0 0
- added joint base_to_camera_link: type fixed, parent base_link, child camera_link, origin xyz=0.045332 0.117283 -0.193859 rpy=0 0 0
- added joint base_to_laser_frame: type fixed, parent base_link, child laser_frame, origin xyz=-0.020598 0.093630 -0.074205 rpy=0 0 0
- added joint base_to_mocap_led_0: type fixed, parent base_link, child mocap_led_0, origin xyz=-0.040 -0.060 0.160 rpy=0 0 0
- added joint base_to_mocap_led_1: type fixed, parent base_link, child mocap_led_1, origin xyz=0.040 -0.060 0.160 rpy=0 0 0
- added joint base_to_mocap_led_2: type fixed, parent base_link, child mocap_led_2, origin xyz=-0.040 0.000 0.160 rpy=0 0 0
- added joint base_to_mocap_led_3: type fixed, parent base_link, child mocap_led_3, origin xyz=0.040 0.000 0.160 rpy=0 0 0
- added joint base_to_mocap_led_4: type fixed, parent base_link, child mocap_led_4, origin xyz=-0.040 0.060 0.160 rpy=0 0 0
- added joint base_to_mocap_led_5: type fixed, parent base_link, child mocap_led_5, origin xyz=0.040 0.060 0.160 rpy=0 0 0
- added joint base_to_mocap_led_6: type fixed, parent base_link, child mocap_led_6, origin xyz=-0.080 0.000 0.190 rpy=0 0 0
- added joint base_to_mocap_led_7: type fixed, parent base_link, child mocap_led_7, origin xyz=0.080 0.000 0.190 rpy=0 0 0
- added joint camera_color_frame_to_optical: type fixed, parent camera_color_frame, child camera_color_optical_frame, origin xyz=0 0 0 rpy=-1.57079632679 0 -1.57079632679
- added joint camera_color_optical_to_camera_optical_frame: type fixed, parent camera_color_optical_frame, child camera_optical_frame, origin xyz=0 0 0 rpy=0 0 0
- added joint camera_depth_frame_to_optical: type fixed, parent camera_depth_frame, child camera_depth_optical_frame, origin xyz=0 0 0 rpy=-1.57079632679 0 -1.57079632679
- added joint camera_link_to_color_frame: type fixed, parent camera_link, child camera_color_frame, origin xyz=0 0 0 rpy=0 0 0
- added joint camera_link_to_depth_frame: type fixed, parent camera_link, child camera_depth_frame, origin xyz=0 0 0 rpy=0 0 0
- added joint laser_frame_to_lidar_link: type fixed, parent laser_frame, child lidar_link, origin xyz=0 0 0 rpy=0 0 0

Commit message: Prepare coursework submission

File: catkin_ws/src/robot_description/urdf/assembly.urdf (robot description, URDF)
Before this commit: robot myagv_assembly, 19 links, 18 joints
Joints:
- joint base_to_assembly_mesh: origin xyz=0.299832 -0.024717 -0.033859 rpy=0 0 0 -> xyz=0.033859 -0.299832 -0.024717 rpy=1.57079632679 0 -1.57079632679
- joint base_to_camera_link: origin xyz=0.045332 0.117283 -0.193859 rpy=0 0 0 -> xyz=0.193859 -0.045332 0.117283 rpy=0 0 0
- joint base_to_laser_frame: origin xyz=-0.020598 0.093630 -0.074205 rpy=0 0 0 -> xyz=0.074205 0.020598 0.093630 rpy=0 0 0
